File: Varity60.kicad_pcb (KiCad board)
At the start: 2 copper layers, 284.7 x 117.2 mm, 73 parts, among them SW1 Rotary_Encoder_Switch

Commit message: pivot MCU
Parts:
- added D1: 1N4148W, Diode_SMD:D_SOD-123, F.Cu at (76.7, 96.1)
- added D10: 1N4148W, Diode_SMD:D_SOD-123, F.Cu at (105.3, 172.5)
- added D11: 1N4148W, Diode_SMD:D_SOD-123, F.Cu at (114.9, 96.1)
- added D12: 1N4148W, Diode_SMD:D_SOD-123, F.Cu at (124.5, 115.3)
- added D13: 1N4148W, Diode_SMD:D_SOD-123, F.Cu at (129.2, 134.4)
- added D14: 1N4148W, Diode_SMD:D_SOD-123, F.Cu at (138.7, 153.4)
- added D15: 1N4148W, Diode_SMD:D_SOD-123, F.Cu at (129.2, 172.5)
- added D16: 1N4148W, Diode_SMD:D_SOD-123, F.Cu at (133.9, 96.3)
- added D17: 1N4148W, Diode_SMD:D_SOD-123, F.Cu at (143.4, 115.2)
- added D18: 1N4148W, Diode_SMD:D_SOD-123, F.Cu at (148.1, 134.4)
- added D19: 1N4148W, Diode_SMD:D_SOD-123, F.Cu at (157.6, 153.3)
- added D2: 1N4148W, Diode_SMD:D_SOD-123, F.Cu at (81.4, 115.3)
- added D20: 1N4148W, Diode_SMD:D_SOD-123, F.Cu at (153.0, 96.1)
- added D21: 1N4148W, Diode_SMD:D_SOD-123, F.Cu at (162.4, 115.2)
- added D22: 1N4148W, Diode_SMD:D_SOD-123, F.Cu at (167.1, 134.2)
- added D23: 1N4148W, Diode_SMD:D_SOD-123, F.Cu at (176.7, 153.4)
- added D24: 1N4148W, Diode_SMD:D_SOD-123, F.Cu at (172.0, 96.3)
- added D25: 1N4148W, Diode_SMD:D_SOD-123, F.Cu at (181.5, 115.3)
- added D26: 1N4148W, Diode_SMD:D_SOD-123, F.Cu at (186.3, 134.2)
- added D27: 1N4148W, Diode_SMD:D_SOD-123, F.Cu at (195.8, 153.3)
- added D28: 1N4148W, Diode_SMD:D_SOD-123, F.Cu at (191.1, 96.1)
- added D29: 1N4148W, Diode_SMD:D_SOD-123, F.Cu at (200.4, 115.1)
- added D3: 1N4148W, Diode_SMD:D_SOD-123, F.Cu at (83.8, 134.4)
- added D30: 1N4148W, Diode_SMD:D_SOD-123, F.Cu at (205.2, 134.2)
- added D31: 1N4148W, Diode_SMD:D_SOD-123, F.Cu at (214.6, 153.2)
- added D32: 1N4148W, Diode_SMD:D_SOD-123, F.Cu at (200.4, 172.2)
- added D33: 1N4148W, Diode_SMD:D_SOD-123, F.Cu at (210.1, 96.1)
- added D34: 1N4148W, Diode_SMD:D_SOD-123, F.Cu at (219.6, 115.1)
- added D35: 1N4148W, Diode_SMD:D_SOD-123, F.Cu at (224.3, 134.1)
- added D36: 1N4148W, Diode_SMD:D_SOD-123, F.Cu at (233.8, 153.3)
- added D37: 1N4148W, Diode_SMD:D_SOD-123, F.Cu at (229.0, 96.1)
- added D38: 1N4148W, Diode_SMD:D_SOD-123, F.Cu at (238.5, 115.2)
- added D39: 1N4148W, Diode_SMD:D_SOD-123, F.Cu at (243.3, 134.2)
- added D4: 1N4148W, Diode_SMD:D_SOD-123, F.Cu at (88.8, 153.3)
- added D40: 1N4148W, Diode_SMD:D_SOD-123, F.Cu at (252.7, 153.4)
- added D41: 1N4148W, Diode_SMD:D_SOD-123, F.Cu at (248.2, 96.1)
- added D42: 1N4148W, Diode_SMD:D_SOD-123, F.Cu at (257.6, 115.3)
- added D43: 1N4148W, Diode_SMD:D_SOD-123, F.Cu at (262.5, 134.4)
- added D44: 1N4148W, Diode_SMD:D_SOD-123, F.Cu at (272.0, 153.4)
- added D45: 1N4148W, Diode_SMD:D_SOD-123, F.Cu at (271.7, 172.3)
- added D46: 1N4148W, Diode_SMD:D_SOD-123, F.Cu at (267.2, 96.1)
- added D47: 1N4148W, Diode_SMD:D_SOD-123, F.Cu at (276.6, 115.3)
- added D48: 1N4148W, Diode_SMD:D_SOD-123, F.Cu at (281.4, 134.4)
- added D49: 1N4148W, Diode_SMD:D_SOD-123, F.Cu at (291.1, 153.3)
- added D5: 1N4148W, Diode_SMD:D_SOD-123, F.Cu at (81.5, 172.3)
- added D50: 1N4148W, Diode_SMD:D_SOD-123, F.Cu at (295.9, 172.6)
- added D51: 1N4148W, Diode_SMD:D_SOD-123, F.Cu at (286.3, 96.1)
- added D52: 1N4148W, Diode_SMD:D_SOD-123, F.Cu at (295.5, 115.2)
- added D53: 1N4148W, Diode_SMD:D_SOD-123, F.Cu at (300.4, 134.2)
- added D54: 1N4148W, Diode_SMD:D_SOD-123, F.Cu at (317.4, 153.4)
- added D55: 1N4148W, Diode_SMD:D_SOD-123, F.Cu at (317.1, 172.3)
- added D56: 1N4148W, Diode_SMD:D_SOD-123, F.Cu at (305.3, 96.1)
- added D57: 1N4148W, Diode_SMD:D_SOD-123, F.Cu at (314.7, 115.2)
- added D58: 1N4148W, Diode_SMD:D_SOD-123, F.Cu at (324.5, 96.3)
- added D59: 1N4148W, Diode_SMD:D_SOD-123, F.Cu at (338.8, 115.3)
- added D6: 1N4148W, Diode_SMD:D_SOD-123, F.Cu at (95.6, 96.0)
- added D60: 1N4148W, Diode_SMD:D_SOD-123, F.Cu at (331.5, 134.2)
- added D61: 1N4148W, Diode_SMD:D_SOD-123, F.Cu at (343.3, 153.3)
- added D62: 1N4148W, Diode_SMD:D_SOD-123, F.Cu at (340.7, 172.3)
- added D63: 1N4148W, Diode_SMD:D_SOD-123, F.Cu at (343.4, 96.3)
- added D7: 1N4148W, Diode_SMD:D_SOD-123, F.Cu at (105.3, 115.3)
- added D8: 1N4148W, Diode_SMD:D_SOD-123, F.Cu at (109.9, 134.2)
- added D9: 1N4148W, Diode_SMD:D_SOD-123, F.Cu at (119.6, 153.2)
- added U1: ChinaBluePill, chinabluepill:ChinaBluePill, F.Cu at (296.2, 62.4)
Connections:
- 15MXLALT1 pad 2: Net-(15MXLALT1-Pad2) -> Net-(125MXLALT1-Pad2)
- 15MXRALT2 pad 2: Net-(15MXRALT2-Pad2) -> Net-(125MXRATL1-Pad2)
- 15MXRCTRL1 pad 2: Net-(15MXRCTRL1-Pad2) -> Net-(125MXLCTRL1-Pad2)
- 15MXRCTRL2 pad 2: Net-(15MXRCTRL2-Pad2) -> Net-(125MXRCTRL1-Pad2)
- 175MXSTCPS1 pad 2: Net-(175MXSTCPS1-Pad2) -> Net-(175MXCPS1-Pad2)
- 6MXSPC1 pad 2: Net-(6MXSPC1-Pad2) -> Net-(6.25MXSPC1-Pad2)
- MXLGUI1 pad 2: Net-(MXLGUI1-Pad2) -> Net-(125MXLGUI1-Pad2)
- MXRGUI1 pad 2: Net-(MXRGUI1-Pad2) -> Net-(125MXRGUI1-Pad2)
- MXRMN1 pad 2: Net-(MXRMN1-Pad2) -> Net-(125MXRMENU1-Pad2)

Commit message: done wiring etc
Parts:
- removed 15MXRCTRL1: MX-NoLED, MX_Only:MXOnly-1.5U-Hotswap-AntiShear
- added 15MXLCTRL1: MX-NoLED, MX_Only:MXOnly-1.5U-Hotswap-AntiShear, F.Cu at (71.4, 171.4)
- added D64: 1N4148W, Diode_SMD:D_SOD-123, B.Cu at (59.9, 82.2)
- added J1: OLED, Connector_PinSocket_2.54mm:PinSocket_1x04_P2.54mm_Vertical, F.Cu at (285.5, 77.6)
- 6MXSPC1: footprint MX_Only:MXOnly-6U-Centered-ReversedStabilizers-Hotswap-AntiShear -> MX_Only:MXOnly-6U-ReversedStabilizers-NoLED-HotSwap-AntiShear
- D1, D10, D11, D12, D13, D14, D15, D16, D17, D18, D19, D2, D20, D21, D22, D23, D24, D25, D26, D27, D28, D29, D3, D30, D31, D32, D33, D34, D35, D36, D37, D38, D39, D4, D40, D41, D42, D43, D44, D45, D46, D47, D48, D49, D5, D50, D51, D52, D53, D54, D55, D56, D57, D58, D59, D6, D60, D61, D62, D63, D7, D8, D9: moved to B.Cu
- moved 6MXSPC1 15.1 mm to (181.0, 171.4)
- moved MX6 6.96 mm to (181.0, 95.2)
- moved 175MXRSFT1 6.74 mm to (307.2, 152.4)
- moved MXEQL1 6.74 mm to (295.3, 95.2)
- moved MXC1 6.74 mm to (147.6, 152.4)
- moved MXLNGL1 6.74 mm to (242.9, 152.4)
- moved MXN1 6.74 mm to (204.8, 152.4)
- moved 125MXRATL1 6.74 mm to (259.6, 171.4)
- moved 125MXRCTRL1 6.74 mm to (331.0, 171.4)
- moved 125MXRGUI1 6.74 mm to (283.4, 171.4)
- moved 125MXRMENU1 6.74 mm to (307.2, 171.4)
- moved MXCLN1 6.74 mm to (271.5, 133.3)
- moved 225MXLSFT1 6.74 mm to (78.6, 152.4)
- moved MX8 6.74 mm to (219.1, 95.2)
- moved MXE1 6.74 mm to (133.3, 114.3)
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Connections:
- net Net-(U1-Pad5V) renamed +5V
- 125MXLALT1 pad 1: Net-(125MXLALT1-Pad1) -> COL2
- 125MXLCTRL1 pad 1: Net-(125MXLCTRL1-Pad1) -> COL0
- 125MXLGUI1 pad 1: Net-(125MXLGUI1-Pad1) -> COL1
- 125MXRATL1 pad 1: Net-(125MXRATL1-Pad1) -> COL10
- 125MXRCTRL1 pad 1: Net-(125MXRCTRL1-Pad1) -> COL13
- 125MXRGUI1 pad 1: Net-(125MXRGUI1-Pad1) -> COL11
- 125MXRMENU1 pad 1: Net-(125MXRMENU1-Pad1) -> COL12
- 15MXBSLSH1 pad 1: Net-(15MXBSLSH1-Pad1) -> COL13
- 15MXLALT1 pad 1: Net-(15MXLALT1-Pad1) -> COL2
- 15MXRALT2 pad 1: Net-(15MXRALT2-Pad1) -> COL10
- 15MXRCTRL2 pad 1: Net-(15MXRCTRL2-Pad1) -> COL13
- 15MXTab1 pad 1: Net-(15MXTab1-Pad1) -> COL0
- 175MXCPS1 pad 1: Net-(175MXCPS1-Pad1) -> COL0
- 175MXRSFT1 pad 1: Net-(175MXRSFT1-Pad1) -> COL11
- 175MXSTCPS1 pad 1: Net-(175MXSTCPS1-Pad1) -> COL0
- 225MXENT1 pad 1: Net-(225MXENT1-Pad1) -> COL12
- 225MXLSFT1 pad 1: Net-(225MXLSFT1-Pad1) -> COL0
- 6.25MXSPC1 pad 1: Net-(6.25MXSPC1-Pad1) -> COL6
- 6MXSPC1 pad 1: Net-(6MXSPC1-Pad1) -> COL6
- D1 pad 1: Net-(D1-Pad1) -> ROW0
- D10 pad 1: Net-(D10-Pad1) -> ROW4
- D11 pad 1: Net-(D11-Pad1) -> ROW0
- D12 pad 1: Net-(D12-Pad1) -> ROW1
- D13 pad 1: Net-(D13-Pad1) -> ROW2
- D14 pad 1: Net-(D14-Pad1) -> ROW3
- D15 pad 1: Net-(D15-Pad1) -> ROW4
- D16 pad 1: Net-(D16-Pad1) -> ROW0
- D17 pad 1: Net-(D17-Pad1) -> ROW1
- D18 pad 1: Net-(D18-Pad1) -> ROW2
- D19 pad 1: Net-(D19-Pad1) -> ROW3
- D2 pad 1: Net-(D2-Pad1) -> ROW1
- D20 pad 1: Net-(D20-Pad1) -> ROW0
- D21 pad 1: Net-(D21-Pad1) -> ROW1
- D22 pad 1: Net-(D22-Pad1) -> ROW2
- D23 pad 1: Net-(D23-Pad1) -> ROW3
- D24 pad 1: Net-(D24-Pad1) -> ROW0
- D25 pad 1: Net-(D25-Pad1) -> ROW1
- D26 pad 1: Net-(D26-Pad1) -> ROW2
- D27 pad 1: Net-(D27-Pad1) -> ROW3
- D28 pad 1: Net-(D28-Pad1) -> ROW0
- D29 pad 1: Net-(D29-Pad1) -> ROW1
- D3 pad 1: Net-(D3-Pad1) -> ROW2
- D30 pad 1: Net-(D30-Pad1) -> ROW2
- D31 pad 1: Net-(D31-Pad1) -> ROW3
- D32 pad 1: Net-(D32-Pad1) -> ROW4
- D33 pad 1: Net-(D33-Pad1) -> ROW0
- D34 pad 1: Net-(D34-Pad1) -> ROW1
- D35 pad 1: Net-(D35-Pad1) -> ROW2
- D36 pad 1: Net-(D36-Pad1) -> ROW3
- D37 pad 1: Net-(D37-Pad1) -> ROW0
- D38 pad 1: Net-(D38-Pad1) -> ROW1
- D39 pad 1: Net-(D39-Pad1) -> ROW2
- D4 pad 1: Net-(D4-Pad1) -> ROW3
- D40 pad 1: Net-(D40-Pad1) -> ROW3
- D41 pad 1: Net-(D41-Pad1) -> ROW0
- D42 pad 1: Net-(D42-Pad1) -> ROW1
- D43 pad 1: Net-(D43-Pad1) -> ROW2
- D44 pad 1: Net-(D44-Pad1) -> ROW3
- D45 pad 1: Net-(D45-Pad1) -> ROW4
- D46 pad 1: Net-(D46-Pad1) -> ROW0
- D47 pad 1: Net-(D47-Pad1) -> ROW1
- D48 pad 1: Net-(D48-Pad1) -> ROW2
- D49 pad 1: Net-(D49-Pad1) -> ROW3
- D5 pad 1: Net-(D5-Pad1) -> ROW4
- D50 pad 1: Net-(D50-Pad1) -> ROW4
- D51 pad 1: Net-(D51-Pad1) -> ROW0
- D52 pad 1: Net-(D52-Pad1) -> ROW1
- D53 pad 1: Net-(D53-Pad1) -> ROW2
- D54 pad 1: Net-(D54-Pad1) -> ROW3
- D55 pad 1: Net-(D55-Pad1) -> ROW4
- D56 pad 1: Net-(D56-Pad1) -> ROW0
- D57 pad 1: Net-(D57-Pad1) -> ROW1
- D58 pad 1: Net-(D58-Pad1) -> ROW0
- D59 pad 1: Net-(D59-Pad1) -> ROW1
- D6 pad 1: Net-(D6-Pad1) -> ROW0
- D60 pad 1: Net-(D60-Pad1) -> ROW2
- D61 pad 1: Net-(D61-Pad1) -> ROW3
- D62 pad 1: Net-(D62-Pad1) -> ROW4
- D63 pad 1: Net-(D63-Pad1) -> ROW2
- D7 pad 1: Net-(D7-Pad1) -> ROW1
- D8 pad 1: Net-(D8-Pad1) -> ROW2
- D9 pad 1: Net-(D9-Pad1) -> ROW3
- MX0 pad 1: Net-(MX0-Pad1) -> COL10
- MX1 pad 1: Net-(MX1-Pad1) -> COL1
- MX2 pad 1: Net-(MX2-Pad1) -> COL2
- MX3 pad 1: Net-(MX3-Pad1) -> COL3
- MX4 pad 1: Net-(MX4-Pad1) -> COL4
- MX5 pad 1: Net-(MX5-Pad1) -> COL5
- MX6 pad 1: Net-(MX6-Pad1) -> COL6
- MX7 pad 1: Net-(MX7-Pad1) -> COL7
- MX8 pad 1: Net-(MX8-Pad1) -> COL8
- MX9 pad 1: Net-(MX9-Pad1) -> COL9
- MXA1 pad 1: Net-(MXA1-Pad1) -> COL1
- MXB1 pad 1: Net-(MXB1-Pad1) -> COL5
- MXBSPC1 pad 1: Net-(MXBSPC1-Pad1) -> COL13
- MXC1 pad 1: Net-(MXC1-Pad1) -> COL3
- MXCLN1 pad 1: Net-(MXCLN1-Pad1) -> COL10
- MXD1 pad 1: Net-(MXD1-Pad1) -> COL3
- MXDEL1 pad 1: Net-(MXDEL1-Pad1) -> COL13
- MXDSH1 pad 1: Net-(MXDSH1-Pad1) -> COL11
- MXE1 pad 1: Net-(MXE1-Pad1) -> COL3
- MXEQL1 pad 1: Net-(MXEQL1-Pad1) -> COL12
- MXESC1 pad 1: Net-(MXESC1-Pad1) -> COL0
- MXF1 pad 1: Net-(MXF1-Pad1) -> COL4
- MXFN1 pad 1: Net-(MXFN1-Pad1) -> COL12
- MXG1 pad 1: Net-(MXG1-Pad1) -> COL5
- MXH1 pad 1: Net-(MXH1-Pad1) -> COL6
- MXI1 pad 1: Net-(MXI1-Pad1) -> COL8
- MXJ1 pad 1: Net-(MXJ1-Pad1) -> COL7
- MXK1 pad 1: Net-(MXK1-Pad1) -> COL8
- MXL1 pad 1: Net-(MXL1-Pad1) -> COL9
- MXLBRAC1 pad 1: Net-(MXLBRAC1-Pad1) -> COL11
- MXLGUI1 pad 1: Net-(MXLGUI1-Pad1) -> COL1
- MXLNGL1 pad 1: Net-(MXLNGL1-Pad1) -> COL8
- MXM1 pad 1: Net-(MXM1-Pad1) -> COL7
- MXN1 pad 1: Net-(MXN1-Pad1) -> COL6
- MXO1 pad 1: Net-(MXO1-Pad1) -> COL9
- MXP1 pad 1: Net-(MXP1-Pad1) -> COL10
- MXQ1 pad 1: Net-(MXQ1-Pad1) -> COL1
- MXQUOT1 pad 1: Net-(MXQUOT1-Pad1) -> COL11
- MXR1 pad 1: Net-(MXR1-Pad1) -> COL4
- MXRBRAC1 pad 1: Net-(MXRBRAC1-Pad1) -> COL12
- MXRGUI1 pad 1: Net-(MXRGUI1-Pad1) -> COL11
- MXRMN1 pad 1: Net-(MXRMN1-Pad1) -> COL12
- MXRNGL1 pad 1: Net-(MXRNGL1-Pad1) -> COL9
- MXS1 pad 1: Net-(MXS1-Pad1) -> COL2
- MXSLSH1 pad 1: Net-(MXSLSH1-Pad1) -> COL10
- MXT1 pad 1: Net-(MXT1-Pad1) -> COL5
- MXU1 pad 1: Net-(MXU1-Pad1) -> COL7
- MXV1 pad 1: Net-(MXV1-Pad1) -> COL4
- MXW1 pad 1: Net-(MXW1-Pad1) -> COL2
- MXX1 pad 1: Net-(MXX1-Pad1) -> COL2
- MXY1 pad 1: Net-(MXY1-Pad1) -> COL6
- MXZ1 pad 1: Net-(MXZ1-Pad1) -> COL1
- SW1 pad A: Net-(SW1-PadA) -> ENCA
- SW1 pad B: Net-(SW1-PadB) -> ENCB
- SW1 pad C: Net-(SW1-PadC) -> GND
- SW1 pad S1: Net-(SW1-PadS1) -> COL3
- SW1 pad S2: Net-(SW1-PadS2) -> SWE2
- U1 pad 3V3: Net-(U1-Pad3V3) -> +3V3
- U1 pad GND: Net-(U1-PadGND) -> GND
- U1 pad PA0: Net-(U1-PadPA0) -> COL4
- U1 pad PA1: Net-(U1-PadPA1) -> COL5
- U1 pad PA12: Net-(U1-PadPA12) -> ROW4
- U1 pad PA15: Net-(U1-PadPA15) -> ROW3
- U1 pad PA2: Net-(U1-PadPA2) -> COL6
- U1 pad PA3: Net-(U1-PadPA3) -> COL7
- U1 pad PA4: Net-(U1-PadPA4) -> COL8
- U1 pad PA5: Net-(U1-PadPA5) -> COL9
- U1 pad PA6: Net-(U1-PadPA6) -> COL10
- U1 pad PA7: Net-(U1-PadPA7) -> COL11
- U1 pad PB0: Net-(U1-PadPB0) -> COL12
- U1 pad PB1: Net-(U1-PadPB1) -> COL13
- U1 pad PB10: Net-(U1-PadPB10) -> SCL
- U1 pad PB11: Net-(U1-PadPB11) -> SDA
- U1 pad PB12: Net-(U1-PadPB12) -> ENCA
- U1 pad PB13: Net-(U1-PadPB13) -> ENCB
- U1 pad PB3: Net-(U1-PadPB3) -> ROW2
- U1 pad PB4: Net-(U1-PadPB4) -> ROW1
- U1 pad PB5: Net-(U1-PadPB5) -> ROW0
- U1 pad PB6: Net-(U1-PadPB6) -> COL0
- U1 pad PB7: Net-(U1-PadPB7) -> COL1
- U1 pad PB8: Net-(U1-PadPB8) -> COL2
- U1 pad PB9: Net-(U1-PadPB9) -> COL3
Routing:
- net ROW4: track 0.00 -> 504.9 mm
- net COL3: track 0.00 -> 381.8 mm
- net ROW3: track 0.00 -> 367.3 mm
- net COL0: track 0.00 -> 363.7 mm, vias 0 -> 2
- net COL1: track 0.00 -> 345.9 mm
- net ROW2: track 0.00 -> 344.9 mm
- net ROW1: track 0.00 -> 329.4 mm
- net COL2: track 0.00 -> 322.8 mm
- net ROW0: track 0.00 -> 289.7 mm
- net ENCA: track 0.00 -> 281.9 mm
- net ENCB: track 0.00 -> 272.0 mm
- net COL4: track 0.00 -> 241.7 mm
- net COL6: track 0.00 -> 236.0 mm
- net GND: track 0.00 -> 229.3 mm
- net COL5: track 0.00 -> 224.0 mm
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Other:
- board size 284.7 x 117.2 mm -> 292.7 x 123.2 mm
- net class Power added: clearance 0.2, trace_width 0.38, via_dia 0.8, via_drill 0.4
