File: Varity60.sch (KiCad schematic (older format))
At the start: 73 parts, among them SW1 Rotary_Encoder_Switch

Commit message: pivot MCU
Parts:
- added D1, D10, D11, D12, D13, D14, D15, D16, D17, D18, D19, D2, D20, D21, D22, D23, D24, D25, D26, D27, D28, D29, D3, D30, D31, D32, D33, D34, D35, D36, D37, D38, D39, D4, D40, D41, D42, D43, D44, D45, D46, D47, D48, D49, D5, D50, D51, D52, D53, D54, D55, D56, D57, D58, D59, D6, D60, D61, D62, D63, D7, D8, D9: 1N4148W, Diode_SMD:D_SOD-123, symbol Diode:1N4148W
- added J1: OLED, symbol Connector_Generic:Conn_01x04
- added U1: ChinaBluePill, chinabluepill:ChinaBluePill, symbol china_bluepill:ChinaBluePill
Connections:
- net COL0: now reaches MXESC1.1 (COL)
- net COL0: now also 125MXLCTRL1.1 (COL), 15MXRCTRL1.1 (COL), 15MXTab1.1 (COL), 175MXCPS1.1 (COL), 175MXSTCPS1.1 (COL), 225MXLSFT1.1 (COL)
- net at MXESC1.2 (ROW): now also D1.2 (A)
- net COL1: now reaches MX1.1 (COL)
- net COL1: now also 125MXLGUI1.1 (COL), MXA1.1 (COL), MXLGUI1.1 (COL), MXQ1.1 (COL), MXZ1.1 (COL)
- net at MX1.2 (ROW): now also D6.2 (A)
- net COL2: now reaches MX2.1 (COL)
- net COL2: now also 125MXLALT1.1 (COL), 15MXLALT1.1 (COL), MXS1.1 (COL), MXW1.1 (COL), MXX1.1 (COL)
- net at MX2.2 (ROW): now also D11.2 (A)
- net COL3: now reaches MX3.1 (COL)
- net COL3: now also MXC1.1 (COL), MXD1.1 (COL), MXE1.1 (COL)
- net at MX3.2 (ROW): now also D16.2 (A)
- net ROW4: now reaches MX4.1 (COL)
- net ROW4: now also MXF1.1 (COL), MXR1.1 (COL), MXV1.1 (COL), D10.1 (K), D15.1 (K), D32.1 (K), D45.1 (K), D5.1 (K), D50.1 (K), D55.1 (K), D62.1 (K)
- net at MX4.2 (ROW): now also D20.2 (A)
- net ROW5: now reaches MX5.1 (COL)
- net ROW5: now also MXB1.1 (COL), MXG1.1 (COL), MXT1.1 (COL)
- net at MX5.2 (ROW): now also D24.2 (A)
- net ROW6: now reaches MX6.1 (COL)
- net ROW6: now also 6.25MXSPC1.1 (COL), 6MXSPC1.1 (COL), MXH1.1 (COL), MXN1.1 (COL), MXY1.1 (COL)
- net at MX6.2 (ROW): now also D28.2 (A)
- net ROW7: now reaches MX7.1 (COL)
- net ROW7: now also MXJ1.1 (COL), MXM1.1 (COL), MXU1.1 (COL)
- net at MX7.2 (ROW): now also D33.2 (A)
- net ROW8: now reaches MX8.1 (COL)
- net ROW8: now also MXI1.1 (COL), MXK1.1 (COL), MXLNGL1.1 (COL)
- net at MX8.2 (ROW): now also D37.2 (A)
- net ROW9: now reaches MX9.1 (COL)
- net ROW9: now also MXL1.1 (COL), MXO1.1 (COL), MXRNGL1.1 (COL)
- net at MX9.2 (ROW): now also D41.2 (A)
- net ROW10: now reaches MX0.1 (COL)
- net ROW10: now also 125MXRATL1.1 (COL), 15MXRALT2.1 (COL), MXCLN1.1 (COL), MXP1.1 (COL), MXSLSH1.1 (COL)
- net at MX0.2 (ROW): now also D46.2 (A)
- net ROW12: now reaches MXEQL1.1 (COL)
- net ROW12: now also 125MXRMENU1.1 (COL), 225MXENT1.1 (COL), MXFN1.1 (COL), MXRBRAC1.1 (COL), MXRMN1.1 (COL)
- net at MXEQL1.2 (ROW): now also D56.2 (A)
- net ROW13: now reaches MXBSPC1.1 (COL)
- net ROW13: now also 125MXRCTRL1.1 (COL), 15MXBSLSH1.1 (COL), 15MXRCTRL2.1 (COL), MXDEL1.1 (COL)
- net at MXBSPC1.2 (ROW): now also D58.2 (A)
- net at 15MXTab1.2 (ROW): now also D2.2 (A)
- net at MXQ1.2 (ROW): now also D7.2 (A)
- net at MXW1.2 (ROW): now also D12.2 (A)
- net at MXE1.2 (ROW): now also D17.2 (A)
- net at MXR1.2 (ROW): now also D21.2 (A)
- net at MXT1.2 (ROW): now also D25.2 (A)
- net at MXY1.2 (ROW): now also D29.2 (A)
- net at MXU1.2 (ROW): now also D34.2 (A)
- net at MXI1.2 (ROW): now also D38.2 (A)
- net at MXO1.2 (ROW): now also D42.2 (A)
- net at MXP1.2 (ROW): now also D47.2 (A)
- net ROW11: now reaches MXLBRAC1.1 (COL)
- net ROW11: now also 125MXRGUI1.1 (COL), 175MXRSFT1.1 (COL), MXDSH1.1 (COL), MXQUOT1.1 (COL), MXRGUI1.1 (COL)
- net at MXLBRAC1.2 (ROW): now also D52.2 (A)
- net at MXRBRAC1.2 (ROW): now also D57.2 (A)
- net at 175MXCPS1.2 (ROW): now also 175MXSTCPS1.2 (ROW), D3.2 (A)
- net at MXA1.2 (ROW): now also D8.2 (A)
- net at MXS1.2 (ROW): now also D13.2 (A)
- net at MXD1.2 (ROW): now also D18.2 (A)
- net at MXF1.2 (ROW): now also D22.2 (A)
- net at MXG1.2 (ROW): now also D26.2 (A)
- net at MXH1.2 (ROW): now also D30.2 (A)
- net at MXJ1.2 (ROW): now also D35.2 (A)
- net at MXK1.2 (ROW): now also D39.2 (A)
- net at MXL1.2 (ROW): now also D43.2 (A)
- net at MXCLN1.2 (ROW): now also D48.2 (A)
- net at MXQUOT1.2 (ROW): now also D53.2 (A)
- net at MXZ1.2 (ROW): now also D9.2 (A)
- net at MXX1.2 (ROW): now also D14.2 (A)
- net at MXC1.2 (ROW): now also D19.2 (A)
- net at MXV1.2 (ROW): now also D23.2 (A)
- net at MXB1.2 (ROW): now also D27.2 (A)
- net at MXN1.2 (ROW): now also D31.2 (A)
- net at MXM1.2 (ROW): now also D36.2 (A)
- net at MXLNGL1.2 (ROW): now also D40.2 (A)
- net at MXRNGL1.2 (ROW): now also D44.2 (A)
- net at MXSLSH1.2 (ROW): now also D49.2 (A)
- net at 175MXRSFT1.2 (ROW): now also D54.2 (A)
- net at 125MXLCTRL1.2 (ROW): now also 15MXRCTRL1.2 (ROW), D5.2 (A)
- net at 125MXLGUI1.2 (ROW): now also MXLGUI1.2 (ROW), D10.2 (A)
- net at 125MXLALT1.2 (ROW): now also 15MXLALT1.2 (ROW), D15.2 (A)
- net at 125MXRATL1.2 (ROW): now also 15MXRALT2.2 (ROW), D45.2 (A)
- net at 125MXRGUI1.2 (ROW): now also MXRGUI1.2 (ROW), D50.2 (A)
- net at 125MXRMENU1.2 (ROW): now also MXRMN1.2 (ROW), D55.2 (A)
- net at 15MXBSLSH1.2 (ROW): now also D59.2 (A)
- net at MXFN1.2 (ROW): now also D61.2 (A)
- net at 125MXRCTRL1.2 (ROW): now also 15MXRCTRL2.2 (ROW), D62.2 (A)
- net at MXDEL1.2 (ROW): now also D63.2 (A)
- net at 225MXENT1.2 (ROW): now also D60.2 (A)
- net at 225MXLSFT1.2 (ROW): now also D4.2 (A)
- net at 6.25MXSPC1.2 (ROW): now also 6MXSPC1.2 (ROW), D32.2 (A)
- net at MXDSH1.2 (ROW): now also D51.2 (A)
- new net ROW0: D1.1 (K), D11.1 (K), D16.1 (K), D20.1 (K), D24.1 (K), D28.1 (K), D33.1 (K), D37.1 (K), D41.1 (K), D46.1 (K), D51.1 (K), D56.1 (K), D58.1 (K), D6.1 (K)
- new net ROW1: D12.1 (K), D17.1 (K), D2.1 (K), D21.1 (K), D25.1 (K), D29.1 (K), D34.1 (K), D38.1 (K), D42.1 (K), D47.1 (K), D52.1 (K), D57.1 (K), D59.1 (K), D7.1 (K)
- new net ROW2: D13.1 (K), D18.1 (K), D22.1 (K), D26.1 (K), D3.1 (K), D30.1 (K), D35.1 (K), D39.1 (K), D43.1 (K), D48.1 (K), D53.1 (K), D60.1 (K), D63.1 (K), D8.1 (K)
- new net ROW3: D14.1 (K), D19.1 (K), D23.1 (K), D27.1 (K), D31.1 (K), D36.1 (K), D4.1 (K), D40.1 (K), D44.1 (K), D49.1 (K), D54.1 (K), D61.1 (K), D9.1 (K)
Other:
- moved on the sheet: 125MXLALT1, 125MXLCTRL1, 125MXLGUI1, 125MXRATL1, 125MXRCTRL1, 125MXRGUI1, 125MXRMENU1, 15MXBSLSH1, 15MXLALT1, 15MXRALT2, 15MXRCTRL1, 15MXRCTRL2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

Commit message: done wiring etc
Parts:
- added D64: 1N4148W, Diode_SMD:D_SOD-123, symbol Diode:1N4148W
- 6MXSPC1: footprint MX_Only:MXOnly-6U-Centered-ReversedStabilizers-Hotswap-AntiShear -> MX_Only:MXOnly-6U-ReversedStabilizers-NoLED-HotSwap-AntiShear
- J1: footprint (none) -> Connector_PinSocket_2.54mm:PinSocket_1x04_P2.54mm_Vertical
- renumbered 15MXRCTRL1 to 15MXLCTRL1
Connections:
- net ROW10 is gone; now on net COL10: 125MXRATL1.1 (COL), 15MXRALT2.1 (COL), MX0.1 (COL), MXCLN1.1 (COL), MXP1.1 (COL), MXSLSH1.1 (COL)
- net ROW11 is gone; now on net COL11: 125MXRGUI1.1 (COL), 175MXRSFT1.1 (COL), MXDSH1.1 (COL), MXLBRAC1.1 (COL), MXQUOT1.1 (COL), MXRGUI1.1 (COL)
- net ROW12 is gone; now on net COL12: 125MXRMENU1.1 (COL), 225MXENT1.1 (COL), MXEQL1.1 (COL), MXFN1.1 (COL), MXRBRAC1.1 (COL), MXRMN1.1 (COL)
- net ROW13 is gone; now on net COL13: 125MXRCTRL1.1 (COL), 15MXBSLSH1.1 (COL), 15MXRCTRL2.1 (COL), MXBSPC1.1 (COL), MXDEL1.1 (COL)
- net ROW5 is gone; now on net COL5: MX5.1 (COL), MXB1.1 (COL), MXG1.1 (COL), MXT1.1 (COL)
- net ROW6 is gone; now on net COL6: 6.25MXSPC1.1 (COL), 6MXSPC1.1 (COL), MX6.1 (COL), MXH1.1 (COL), MXN1.1 (COL), MXY1.1 (COL)
- net ROW7 is gone; now on net COL7: MX7.1 (COL), MXJ1.1 (COL), MXM1.1 (COL), MXU1.1 (COL)
- net ROW8 is gone; now on net COL8: MX8.1 (COL), MXI1.1 (COL), MXK1.1 (COL), MXLNGL1.1 (COL)
- net ROW9 is gone; now on net COL9: MX9.1 (COL), MXL1.1 (COL), MXO1.1 (COL), MXRNGL1.1 (COL)
- net COL0: now also U1.PB6
- net COL1: now also U1.PB7
- net COL2: now also U1.PB8
- net COL3: now also SW1.S1, U1.PB9
- net ROW0: now also U1.PB5
- net ROW1: now also U1.PB4
- net ROW2: now also U1.PB3
- net ROW3: now also U1.PA15
- net ROW4: now also U1.PA12, D64.1 (K); no longer MX4.1 (COL), MXF1.1 (COL), MXR1.1 (COL), MXV1.1 (COL)
- net GND: now reaches J1.1 (Pin_1)
- net GND: now also SW1.C, U1.GND
- net +3V3: now reaches J1.2 (Pin_2)
- net +3V3: now also U1.3V3
- net SCL: now reaches J1.3 (Pin_3)
- net SCL: now also U1.PB10
- net SDA: now reaches J1.4 (Pin_4)
- net SDA: now also U1.PB11
- net ENCA: now reaches SW1.A
- net ENCA: now also U1.PB12
- net ENCB: now reaches SW1.B
- net ENCB: now also U1.PB13
- net SWE2: now reaches SW1.S2
- net SWE2: now also D64.2 (A)
- net +5V: now reaches U1.5V
- net COL4: now reaches U1.PA0
- net COL4: now also MX4.1 (COL), MXF1.1 (COL), MXR1.1 (COL), MXV1.1 (COL)
- net COL5: now reaches U1.PA1
- net COL6: now reaches U1.PA2
- net COL7: now reaches U1.PA3
- net COL8: now reaches U1.PA4
- net COL9: now reaches U1.PA5
- net COL10: now reaches U1.PA6
- net COL11: now reaches U1.PA7
- net COL12: now reaches U1.PB0
- net COL13: now reaches U1.PB1
Other:
- moved on the sheet: J1
Changed lines of the file:
@@
 $EndComp
 $Comp
-L MX_Alps_Hybrid:MX-NoLED 15MXRCTRL1
+L MX_Alps_Hybrid:MX-NoLED 15MXLCTRL1
 U 1 1 5F544C28
 P 2650 7600
-F 0 "15MXRCTRL1" H 2683 7823 60  0000 C CNN
+F 0 "15MXLCTRL1" H 2683 7823 60  0000 C CNN
 F 1 "MX-NoLED" H 2683 7749 20  0000 C CNN
 F 2 "MX_Only:MXOnly-1.5U-Hotswap-AntiShear" H 2025 7575 60  0001 C CNN
@@
 F 0 "6MXSPC1" H 5583 7823 60  0000 C CNN
 F 1 "MX-NoLED" H 5583 7749 20  0000 C CNN
-F 2 "MX_Only:MXOnly-6U-Centered-ReversedStabilizers-Hotswap-AntiShear" H 4925 7575 60  0001 C CNN
+F 2 "MX_Only:MXOnly-6U-ReversedStabilizers-NoLED-HotSwap-AntiShear" H 4925 7575 60  0001 C CNN
 F 3 "" H 4925 7575 60  0001 C CNN
 	1    5550 7600
@@
 F 0 "J1" H 2818 1275 50  0000 C CNN
 F 1 "OLED" H 2818 1366 50  0000 C CNN
-F 2 "" H 2900 1700 50  0001 C CNN
+F 2 "Connector_PinSocket_2.54mm:PinSocket_1x04_P2.54mm_Vertical" H 2900 1700 50  0001 C CNN
 F 3 "~" H 2900 1700 50  0001 C CNN
 	1    2900 1700
-	-1   0    0    1
+	0    -1   -1   0
 $EndComp
 $Comp
@@
 	2000 5350 2600 5350
 Connection ~ 2600 5350
-$Comp
-L china_bluepill:ChinaBluePill U1
-U 1 1 5F531D9D
-P 12400 2550
-F 0 "U1" H 12400 3365 50  0000 C CNN
-F 1 "ChinaBluePill" H 12400 3274 50  0000 C CNN
-F 2 "chinabluepill:ChinaBluePill" H 12400 2550 50  0001 C CNN
-F 3 "" H 12400 2550 50  0001 C CNN
-	1    12400 2550
-	1    0    0    -1
-$EndComp
 Wire Wire Line
 	2800 3000 2800 3450
@@
 	9400 3450 9400 4400
 Connection ~ 9400 4400
-Wire Wire Line
-	9400 4400 9400 5150
 Connection ~ 9400 6800
 Wire Wire Line
@@
 	8800 5950 8800 6800
 Connection ~ 8800 5950
-Wire Wire Line
-	9400 5150 9400 6800
 Connection ~ 9400 5150
 Wire Wire Line
@@
 	3500 7300 3050 7300
 Connection ~ 5500 7300
-Wire Wire Line
-	5500 7300 3500 7300
 Connection ~ 7500 7300
 Wire Wire Line
@@
 COL3
 Text GLabel 4700 3000 1    50   Input ~ 0
+COL4
+Text GLabel 5200 3000 1    50   Input ~ 0
+COL5
+Text GLabel 5700 3000 1    50   Input ~ 0
+COL6
+Text GLabel 6200 3000 1    50   Input ~ 0
+COL7
+Text GLabel 6700 3000 1    50   Input ~ 0
+COL8
+Text GLabel 7200 3000 1    50   Input ~ 0
+COL9
+Text GLabel 7700 3000 1    50   Input ~ 0
+COL10
+Text GLabel 8250 3000 1    50   Input ~ 0
+COL11
+Text GLabel 8800 3000 1    50   Input ~ 0
+COL12
+Text GLabel 9400 3000 1    50   Input ~ 0
+COL13
+Text GLabel 3100 1900 3    50   Input ~ 0
+SDA
+Text GLabel 3000 1900 3    50   Input ~ 0
+SCL
+$Comp
+L power:GND #PWR0101
+U 1 1 5F3EA610
+P 2800 1900
+F 0 "#PWR0101" H 2800 1650 50  0001 C CNN
+F 1 "GND" H 2805 1727 50  0000 C CNN
+F 2 "" H 2800 1900 50  0001 C CNN
+F 3 "" H 2800 1900 50  0001 C CNN
+	1    2800 1900
+	1    0    0    -1
+$EndComp
+Text GLabel 13100 3000 2    50   Input ~ 0
+SDA
+Text GLabel 13100 2900 2    50   Input ~ 0
+SCL
+$Comp
+L power:+3.3V #PWR0102
+U 1 1 5F3ECB4F
+P 2900 1900
+F 0 "#PWR0102" H 2900 1750 50  0001 C CNN
+F 1 "+3.3V" H 2915 2073 50  0000 C CNN
+F 2 "" H 2900 1900 50  0001 C CNN
+F 3 "" H 2900 1900 50  0001 C CNN
+	1    2900 1900
+	-1   0    0    1
+$EndComp
+$Comp
+L power:GND #PWR0103
+U 1 1 5F3EECC0
+P 13100 3800
+F 0 "#PWR0103" H 13100 3550 50  0001 C CNN
+F 1 "GND" H 13105 3627 50  0000 C CNN
+F 2 "" H 13100 3800 50  0001 C CNN
+F 3 "" H 13100 3800 50  0001 C CNN
+	1    13100 3800
+	1    0    0    -1
+$EndComp
+$Comp
+L power:+3.3V #PWR0104
+U 1 1 5F3EF628
+P 11700 3600
+F 0 "#PWR0104" H 11700 3450 50  0001 C CNN
+F 1 "+3.3V" V 11715 3728 50  0000 L CNN
+F 2 "" H 11700 3600 50  0001 C CNN
+F 3 "" H 11700 3600 50  0001 C CNN
+	1    11700 3600
+	0    -1   -1   0
+$EndComp
+$Comp
+L power:GND #PWR0105
+U 1 1 5F3F15F8
+P 4950 1650
+F 0 "#PWR0105" H 4950 1400 50  0001 C CNN
+F 1 "GND" V 4955 1522 50  0000 R CNN
+F 2 "" H 4950 1650 50  0001 C CNN
+F 3 "" H 4950 1650 50  0001 C CNN
+	1    4950 1650
+	0    1    1    0
+$EndComp
+Text GLabel 5550 1550 2    50   Input ~ 0
+SWE1
+Text GLabel 5550 1750 2    50   Input ~ 0
+SWE2
+Text GLabel 4200 6700 0    50   Input ~ 0
+SWE1
+Text GLabel 4000 7000 1    50   Input ~ 0
+SWE2
+$Comp
+L Diode:1N4148W D64
+U 1 1 5F3FC91B
+P 4000 7150
+F 0 "D64" V 4046 7070 50  0000 R CNN
+F 1 "1N4148W" V 3955 7070 50  0000 R CNN
+F 2 "Diode_SMD:D_SOD-123" H 4000 6975 50  0001 C CNN
+F 3 "https://www.vishay.com/docs/85748/1n4148w.pdf" H 4000 7150 50  0001 C CNN
+	1    4000 7150
+	0    -1   -1   0
+$EndComp
+Wire Wire Line
+	9400 4400 9400 5150
+Wire Wire Line
+	3500 7300 4000 7300
+Text GLabel 11700 2000 0    50   Input ~ 0
+COL4
+Text GLabel 11700 2100 0    50   Input ~ 0
+COL5
+Text GLabel 11700 2200 0    50   Input ~ 0
+COL6
+Text GLabel 11700 2300 0    50   Input ~ 0
+COL7
+Text GLabel 11700 2400 0    50   Input ~ 0
+COL8
+Text GLabel 11700 2500 0    50   Input ~ 0
+COL9
+Text GLabel 11700 2600 0    50   Input ~ 0
+COL10
+Text GLabel 11700 2700 0    50   Input ~ 0
+COL11
+Text GLabel 13100 2000 2    50   Input ~ 0
+COL12
+Text GLabel 13100 2100 2    50   Input ~ 0
+COL13
+Text GLabel 4950 1550 0    50   Input ~ 0
+ENCA
+Text GLabel 4950 1750 0    50   Input ~ 0
+ENCB
+Text GLabel 13100 3100 2    50   Input ~ 0
+ENCA
+Text GLabel 13100 3200 2    50   Input ~ 0
+ENCB
+$Comp
+L power:+5V #PWR0106
+U 1 1 5F677427
+P 11700 3700
+F 0 "#PWR0106" H 11700 3550 50  0001 C CNN
+F 1 "+5V" V 11715 3828 50  0000 L CNN
+F 2 "" H 11700 3700 50  0001 C CNN
+F 3 "" H 11700 3700 50  0001 C CNN
+	1    11700 3700
+	0    -1   -1   0
+$EndComp
+Text GLabel 11700 3200 0    50   Input ~ 0
 ROW4
-Text GLabel 5200 3000 1    50   Input ~ 0
-ROW5
-Text GLabel 5700 3000 1    50   Input ~ 0
-ROW6
-Text GLabel 6200 3000 1    50   Input ~ 0
-ROW7
-Text GLabel 6700 3000 1    50   Input ~ 0
-ROW8
-Text GLabel 7200 3000 1    50   Input ~ 0
-ROW9
-Text GLabel 7700 3000 1    50   Input ~ 0
-ROW10
-Text GLabel 8250 3000 1    50   Input ~ 0
-ROW11
-Text GLabel 8800 3000 1    50   Input ~ 0
-ROW12
-Text GLabel 9400 3000 1    50   Input ~ 0
-ROW13
+Text GLabel 11700 3300 0    50   Input ~ 0
+ROW3
+Text GLabel 13100 2200 2    50   Input ~ 0
+ROW2
+Text GLabel 13100 2300 2    50   Input ~ 0
+ROW1
+Text GLabel 13100 2400 2    50   Input ~ 0
+ROW0
+Connection ~ 4000 7300
+Wire Wire Line
+	4000 7300 5500 7300
+Wire Wire Line
+	4200 5950 4200 6700
+Connection ~ 4200 5950
+Wire Wire Line
+	9400 5150 9400 6800
+$Comp
+L china_bluepill:ChinaBluePill U1
+U 1 1 5F531D9D
+P 12400 2550
+F 0 "U1" H 12400 3365 50  0000 C CNN
+F 1 "ChinaBluePill" H 12400 3274 50  0000 C CNN
+F 2 "chinabluepill:ChinaBluePill" H 12400 2550 50  0001 C CNN
+F 3 "" H 12400 2550 50  0001 C CNN
+	1    12400 2550
+	1    0    0    -1
+$EndComp
+Text GLabel 13100 2800 2    50   Input ~ 0
+COL3
+Text GLabel 13100 2700 2    50   Input ~ 0
+COL2
+Text GLabel 13100 2600 2    50   Input ~ 0
+COL1
+Text GLabel 13100 2500 2    50   Input ~ 0
+COL0
 $EndSCHEMATC
