File: Pill60.kicad_pcb (KiCad board)
At the start: 2 copper layers, 292.7 x 123.2 mm, 161 parts, among them J1 OLED, SW1 Rotary_Encoder_Switch, U1 ChinaBluePill

Commit message: connecting some grounds
Routing:
- net GND: track 236.7 -> 309.3 mm, vias 0 -> 4

Commit message: Fix wires and make stuff better
Connections:
- U1 pad PA12: ROW4 -> ROW3
- U1 pad PA15: ROW3 -> ROW2
- U1 pad PB12: ENCA -> ENCB
- U1 pad PB13: ENCB -> ENCA
- U1 pad PB3: ROW2 -> ROW1
- U1 pad PB4: ROW1 -> ROW0
- U1 pad PB5: ROW0 -> ROW4
- U1 pad PB6: COL0 -> COL3
- U1 pad PB7: COL1 -> COL0
- U1 pad PB8: COL2 -> COL1
- U1 pad PB9: COL3 -> COL2
Routing:
- net ROW4: track 516.6 -> 647.7 mm
- net COL2: track 322.8 -> 358.7 mm
- net GND: track 309.3 -> 287.2 mm, vias 4 -> 2
- net ROW0: track 568.5 -> 552.3 mm
- net COL3: track 397.4 -> 389.9 mm
- net ROW1: track 590.6 -> 585.6 mm
- net LED: track 51.0 -> 55.6 mm
- net COL1: track 345.9 -> 350.1 mm
- net ROW3: track 628.8 -> 632.7 mm
- net ROW2: track 643.3 -> 647.1 mm
- net ENCA: track 281.9 -> 278.3 mm
- net COL0: track 363.7 -> 361.2 mm

Commit message: delete more unnecessary ground wire
Routing:
- net GND: track 287.2 -> 1.62 mm, vias 2 -> 0
- net ENCB: track 272.2 -> 274.4 mm
