File: Pill60.kicad_pcb (KiCad board)
At the start: 2 copper layers, 292.7 x 123.2 mm, 161 parts, among them J1 OLED, SW1 Rotary_Encoder_Switch, U1 ChinaBluePill

Commit message: Better wires
Routing:
- net Net-(L6-Pad1): track 65.0 -> 47.1 mm

Commit message: fixed stupid mistake
Routing:
- net Net-(L6-Pad1): track 47.1 -> 65.1 mm
Changed lines of the file:
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@@
     (thickness 1.6)
     (drawings 752)
-    (tracks 692)
+    (tracks 696)
     (zones 0)
     (modules 161)
@@
   (segment (start 311.25 105.22) (end 310.82 105.65) (width 0.38) (layer B.Cu) (net 100))
   (segment (start 330.3 105.22) (end 311.25 105.22) (width 0.38) (layer B.Cu) (net 100))
-  (via (at 330.3 105.22) (size 0.8) (drill 0.4) (layers F.Cu B.Cu) (net 100))
-  (segment (start 340.76 105.22) (end 330.3 105.22) (width 0.38) (layer F.Cu) (net 100))
   (segment (start 344.032001 101.947999) (end 340.76 105.22) (width 0.38) (layer F.Cu) (net 100))
   (segment (start 344.032001 80.797039) (end 344.032001 101.947999) (width 0.38) (layer F.Cu) (net 100))
@@
   (segment (start 299.7 66.11) (end 300.852001 67.262001) (width 0.38) (layer F.Cu) (net 100))
   (segment (start 300.892001 67.262001) (end 312.56498 78.93498) (width 0.38) (layer F.Cu) (net 100))
+  (via (at 337.44 105.22) (size 0.8) (drill 0.4) (layers F.Cu B.Cu) (net 100))
+  (segment (start 330.3 105.22) (end 337.44 105.22) (width 0.38) (layer B.Cu) (net 100))
+  (segment (start 337.44 105.22) (end 340.76 105.22) (width 0.38) (layer F.Cu) (net 100))
   (segment (start 307.32 105.65) (end 306.63 105.65) (width 0.25) (layer B.Cu) (net 101))
   (segment (start 304.88 103.9) (end 274.33 103.9) (width 0.25) (layer B.Cu) (net 101))
@@
   (segment (start 85.51 105.64) (end 84.160737 106.989263) (width 0.25) (layer B.Cu) (net 108))
   (segment (start 84.160737 147.721515) (end 81.17 150.712252) (width 0.25) (layer F.Cu) (net 108))
-  (segment (start 84.160737 135.630737) (end 84.160737 147.721515) (width 0.25) (layer F.Cu) (net 108))
   (segment (start 81.17 150.712252) (end 81.17 153.66) (width 0.25) (layer F.Cu) (net 108))
   (via (at 77.9 159.63) (size 0.8) (drill 0.4) (layers F.Cu B.Cu) (net 108))
@@
   (segment (start 84.160737 106.989263) (end 84.160737 117.758078) (width 0.25) (layer B.Cu) (net 108))
   (segment (start 84.160737 117.758078) (end 84.150883 117.767932) (width 0.25) (layer B.Cu) (net 108))
+  (segment (start 84.150883 135.770883) (end 84.160737 135.780737) (width 0.25) (layer F.Cu) (net 108))
+  (segment (start 84.150883 117.767932) (end 84.150883 135.770883) (width 0.25) (layer F.Cu) (net 108))
+  (segment (start 84.160737 135.630737) (end 84.160737 135.780737) (width 0.25) (layer F.Cu) (net 108))
+  (segment (start 84.160737 135.780737) (end 84.160737 147.721515) (width 0.25) (layer F.Cu) (net 108))
   (segment (start 89.161653 163.553911) (end 91.804424 163.55391) (width 0.25) (layer B.Cu) (net 109))
   (segment (start 85.09 161.05) (end 86.657742 161.05) (width 0.25) (layer B.Cu) (net 109))

Commit message: added more holes for plate and pcb mounting
Parts:
- added H10: Hole, MountingHole:MountingHole_2.2mm_M2, F.Cu at (342.0, 180.5)
- added H8: Hole, MountingHole:MountingHole_2.2mm_M2, F.Cu at (57.8, 180.5)
- added H9: Hole, MountingHole:MountingHole_2.2mm_M2, F.Cu at (249.1, 171.5)
- moved H6 266.9 mm to (316.3, 114.2)
- moved H1 260.9 mm to (86.9, 126.4)
- moved H2 208.0 mm to (294.0, 145.4)
- moved H3 81.0 mm to (279.4, 65.8)
- moved H5 56.6 mm to (317.8, 107.3)
- moved J1 0.08 mm to (285.5, 77.5)
Other:
- board text added: "case hole"
- board text added: "oled hole"
- board text added: "plate hole"
