File: Pill60.kicad_pcb (KiCad board)
At the start: 2 copper layers, 292.7 x 123.2 mm, 164 parts, among them J1 OLED, SW1 Rotary_Encoder_Switch, U1 ChinaBluePill

Commit message: added support for blackpill
Connections:
- U1 pad PA0: COL4 -> Net-(U1-PadPA0)
- U1 pad PA10: Net-(U1-PadPA10) -> COL4
- U1 pad PA11: Net-(U1-PadPA11) -> COL0
- U1 pad PA8: Net-(U1-PadPA8) -> COL3
- U1 pad PB10: SCL -> COL2
- U1 pad PB11: SDA -> COL1
- U1 pad PB12: ENCB -> Net-(U1-PadPB12)
- U1 pad PB13: ENCA -> Net-(U1-PadPB13)
- U1 pad PB6: COL3 -> SCL
- U1 pad PB7: COL0 -> SDA
- U1 pad PB8: COL1 -> ENCB
- U1 pad PB9: COL2 -> ENCA
Routing:
- net ENCB: track 274.3 -> 236.2 mm
- net ENCA: track 278.3 -> 240.2 mm
- net COL1: track 350.1 -> 384.3 mm
- net COL2: track 358.7 -> 392.7 mm
- net COL4: track 243.9 -> 273.0 mm, vias 0 -> 1
- net SDA: track 52.0 -> 24.6 mm
- net COL3: track 389.9 -> 412.7 mm
- net COL0: track 361.2 -> 378.8 mm
- net SCL: track 48.4 -> 34.6 mm

Commit message: changed pin diagram to avoid bad pin
Connections:
- U1 pad PA11: COL0 -> Net-(U1-PadPA11)
- U1 pad PA12: ROW3 -> Net-(U1-PadPA12)
- U1 pad PA8: COL3 -> COL0
- U1 pad PA9: LED -> Net-(U1-PadPA9)
- U1 pad PB13: Net-(U1-PadPB13) -> ROW3
- U1 pad PB14: Net-(U1-PadPB14) -> LED
- U1 pad PB15: Net-(U1-PadPB15) -> COL3
Routing:
- net ROW3: track 632.7 -> 650.3 mm
- net COL0: track 378.8 -> 386.5 mm
- net COL3: track 412.7 -> 415.1 mm
