File: Pill60.sch (KiCad schematic (older format))
At the start: 163 parts, among them J1 OLED, SW1 Rotary_Encoder_Switch, U1 ChinaBluePill

Commit message: update readme and add case files
Parts:
- 175MXCPS1: footprint MX_Only:MXOnly-1.75U-Hotswap -> MX_Only:MXOnly-1.75U-NoLED
- 175MXSTCPS1: footprint MX_Only:MXOnly-1.75U-Hotswap -> MX_Only:MXOnly-1U-NoLED
Changed lines of the file:
@@
 F 0 "175MXSTCPS1" H 2083 5423 60  0000 C CNN
 F 1 "MX-NoLED" H 2083 5349 20  0000 C CNN
-F 2 "MX_Only:MXOnly-1.75U-Hotswap" H 1425 5175 60  0001 C CNN
+F 2 "MX_Only:MXOnly-1U-NoLED" H 1425 5175 60  0001 C CNN
 F 3 "" H 1425 5175 60  0001 C CNN
 	1    2050 5200
@@
 F 0 "175MXCPS1" H 2683 5423 60  0000 C CNN
 F 1 "MX-NoLED" H 2683 5349 20  0000 C CNN
-F 2 "MX_Only:MXOnly-1.75U-Hotswap" H 2025 5175 60  0001 C CNN
+F 2 "MX_Only:MXOnly-1.75U-NoLED" H 2025 5175 60  0001 C CNN
 F 3 "" H 2025 5175 60  0001 C CNN
 	1    2650 5200
